File: ksoloti-power-midi-board.kicad_sch (KiCad schematic)
At the start: 41 parts, among them J1 VIN, J2 DC 9-20V, J3 MIDI_IN, J4 MIDI_OUT, J5 MIDI_THRU, J6 BREAKOUT_CONN, U1 TPS5430DDA, U2 74HC14

Commit message: edits, update cpl and project.db
Other:
- note added: "DC to 5V and MIDI"
- note removed: "DC to 5V and MIDI (detachable subboard)"
Changed lines of the file:
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@@
   (junction (at 175.26 54.61) (diameter 0) (color 0 0 0 0)
   )
+  (junction (at 35.56 54.61) (diameter 0) (color 0 0 0 0)
+  )
   (junction (at 53.34 49.53) (diameter 0) (color 0 0 0 0)
   )
@@
   )
   (junction (at 59.69 63.5) (diameter 0) (color 0 0 0 0)
-  )
-  (junction (at 45.72 52.07) (diameter 0) (color 0 0 0 0)
   )
   (junction (at 252.73 40.64) (diameter 0) (color 0 0 0 0)
@@
     (effects (font (size 1.27 1.27)) (justify left bottom))
   )
-  (text "DC to 5V and MIDI (detachable subboard)" (at 20.32 33.02 0)
+  (text "DC to 5V and MIDI" (at 20.32 33.02 0)
     (effects (font (size 3 3)) (justify left bottom))
   )
@@
     (pin "1")
   )
-  (symbol (lib_id "power:PWR_FLAG") (at 45.72 52.07 270) (unit 1)
-    (in_bom yes) (on_board yes) (fields_autoplaced)
-    (property "Reference" "#FLG02" (id 0) (at 47.625 52.07 0)
-      (effects (font (size 1.27 1.27)) hide)
-    )
-    (property "Value" "PWR_FLAG" (id 1) (at 49.53 52.07 0)
-      (effects (font (size 1.27 1.27)) hide)
-    )
-    (property "Footprint" "" (id 2) (at 45.72 52.07 0)
-      (effects (font (size 1.27 1.27)) hide)
-    )
-    (property "Datasheet" "~" (id 3) (at 45.72 52.07 0)
-      (effects (font (size 1.27 1.27)) hide)
-    )
+  (symbol (lib_id "power:PWR_FLAG") (at 35.56 54.61 270) (unit 1)
+    (in_bom yes) (on_board yes) (fields_autoplaced)
+    (property "Reference" "#FLG02" (id 0) (at 37.465 54.61 0)
+      (effects (font (size 1.27 1.27)) hide)
+    )
+    (property "Value" "PWR_FLAG" (id 1) (at 39.37 54.61 0)
+      (effects (font (size 1.27 1.27)) hide)
+    )
+    (property "Footprint" "" (id 2) (at 35.56 54.61 0)
+      (effects (font (size 1.27 1.27)) hide)
+    )
+    (property "Datasheet" "~" (id 3) (at 35.56 54.61 0)
+      (effects (font (size 1.27 1.27)) hide)
+    )
